File: PCB/MacroPadPro.kicad_sch (KiCad schematic)
At the start: 118 parts, among them J1 Button, J2 Button, SW1 CPG151101S11, SW10 CPG151101S11, SW11 CPG151101S11, SW12 CPG151101S11, SW13 CPG151101S11, SW14 CPG151101S11, SW15 CPG151101S11, SW16 CPG151101S11, SW17 CPG151101S11, SW18 CPG151101S11, SW19 CPG151101S11, SW2 CPG151101S11, SW20 CPG151101S11, SW21 CPG151101S11, SW22 CPG151101S11, SW23 CPG151101S11, SW24 CPG151101S11, SW25 CPG151101S11, SW26 CPG151101S11, SW27 CPG151101S11, SW3 CPG151101S11, SW4 CPG151101S11, SW5 CPG151101S11, SW6 CPG151101S11, SW7 CPG151101S11, SW8 CPG151101S11, SW9 CPG151101S11, U1 ZL6201A33S3, U3 RP2040, Y1 3225-4P 12MHz

Commit message: Updated PCB design to fix GND fault and update BOM components
Parts:
- removed GPIO25_LED1: LED 0402, LED_SMD:LED_0402_1005Metric, symbol Device:LED
- removed GPIO25_RESISTOR1: 1K 0402, Resistor_SMD:R_0402_1005Metric, symbol Device:R
- U1: value ZL6201A33S3 -> AP2210N-3.3TRG1
Other:
- note added: "LED DIODES"
- note added: "RP2040 + Resistors / Capacitors"
- note added: "Switches"
- note removed: "GD25Q40CEIGR is NOT Compatible you need GD25W16* needs to be a multiple of 8 atleast for circuitpython."
- note removed: "Im pretty sure a lot of these W25QXXX Chips are pin compatible Dont quote me on that"
- note removed: "Im unsure if the RP2040 can function with flash larger than 128Mb"
- note removed: "JLCPCB Often has W25Q16FWUXIE in stock but its reccomended as its suposedly only 1.8V although for some reason it works"
- note removed: "Make sure C10 is close to pin 44 of RP2040"
- note removed: "Make sure C3 is close to pin 45 of RP2040"
- note removed: "Make sure R3 and R4 are close to RP2040"
- note removed: "Pin 9 technically doesnt exist its the main central contact under the chip for heat dicipation"
- note removed: "These decoupling capacitors are meant to be put close by each 3.3V pin of the RP2040"
- note removed: "this is for factory testing always pull this to ground"
- moved on the sheet: C1, C10, C11, C12, C13, C14, C15, C16, C2, C3, C4, C5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
